File: pmw3610_pcb.kicad_pcb (KiCad board)
At the start: 2 copper layers, 15.4 x 29.9 mm, 15 parts, among them J1 Conn_01x02, J2 Conn_01x04, U1 PMW3610, U2 TLV74318PDBVR

Commit message: variant of long flex pcb
Parts:
- moved C1 8.80 mm to (149.3, 81.5)
- moved C10 8.80 mm to (155.0, 78.9)
- moved C2 8.80 mm to (151.0, 81.5)
- moved C3 8.80 mm to (146.1, 81.5)
- moved C4 8.80 mm to (152.7, 81.5)
- moved C5 8.80 mm to (147.7, 81.5)
- moved C6 8.80 mm to (154.4, 81.5)
- moved C7 8.80 mm to (156.0, 81.5)
- moved C8 8.80 mm to (147.5, 77.9)
- moved C9 8.80 mm to (155.0, 77.2)
- moved J1 8.80 mm to (144.9, 77.9)
- moved R1 8.80 mm to (144.5, 81.5)
- moved U2 8.80 mm to (150.8, 78.1)
- moved J2 8.80 mm to (155.3, 75.4)
Routing:
- net Net-(U1-+VCSEL): track 33.5 -> 51.1 mm
- net Net-(U1-CN): track 14.8 -> 23.6 mm
- net +1V8: track 23.5 -> 32.3 mm
- net GND: track 59.9 -> 68.8 mm
- net MOTION: track 39.4 -> 48.2 mm
- net SDIO: track 18.4 -> 27.2 mm
- net nCS: track 31.0 -> 39.8 mm
- net SCLK: track 20.6 -> 29.4 mm
- net Net-(U1-VCP): track 22.6 -> 31.4 mm
- net Net-(U1-NRESET): track 17.5 -> 26.3 mm
- net Net-(U1-CP): track 18.5 -> 27.3 mm
- net VIN: track 30.0 -> 38.8 mm
Other:
- board size 15.4 x 29.9 mm -> 15.5 x 38.7 mm
